Commit message: Sprint 3: Continuous wheel joints and first wheel rotation

File: robot_ws/src/orion_description/urdf/links/wheel.xacro (robot description, xacro)
@@ -54,5 +54,5 @@
         <joint
             name="${wheel_name}_joint"
-            type="fixed">
+            type="continuous">
             <parent link="${parent_link}"/>
             <child link="${wheel_name}"/>
@@ -60,4 +60,6 @@
                 xyz="${x} ${y} ${z}"
                 rpy="0 0 0"/>
+           <axis xyz="0 1 0"/>
+	  <dynamics damping="0.2" friction="0.1"/>
         </joint>
     </xacro:macro>
