Commit message: Sprint 3: Launch Gazebo directly from Xacro

File: robot_ws/src/orion_description/urdf/robot/orion.urdf (robot description, URDF)
Before this commit: robot orion, 2 links, 1 joints
Links:
- added link front_left_wheel, mass 1.5; collision cylinder length=0.06 radius=0.12; visual cylinder length=0.06 radius=0.12
- added link front_right_wheel, mass 1.5; collision cylinder length=0.06 radius=0.12; visual cylinder length=0.06 radius=0.12
- added link rear_left_wheel, mass 1.5; collision cylinder length=0.06 radius=0.12; visual cylinder length=0.06 radius=0.12
- added link rear_right_wheel, mass 1.5; collision cylinder length=0.06 radius=0.12; visual cylinder length=0.06 radius=0.12
Joints:
- added joint front_left_wheel_joint: type continuous, parent base_link, child front_left_wheel, origin xyz=0.25 0.26 0.12 rpy=0 0 0, axis 0 1 0
- added joint front_right_wheel_joint: type continuous, parent base_link, child front_right_wheel, origin xyz=0.25 -0.26 0.12 rpy=0 0 0, axis 0 1 0
- added joint rear_left_wheel_joint: type continuous, parent base_link, child rear_left_wheel, origin xyz=-0.25 0.26 0.12 rpy=0 0 0, axis 0 1 0
- added joint rear_right_wheel_joint: type continuous, parent base_link, child rear_right_wheel, origin xyz=-0.25 -0.26 0.12 rpy=0 0 0, axis 0 1 0
